Commit message: added stanbot

File: model/stanbot/stanbot.urdf (robot description, URDF)
Before this commit: robot stanbot, 31 links, 30 joints
Links:
- removed link head_rx
- removed link head_ry
- removed link hip
- removed link left_foot_rx
- removed link left_foot_ry
- added link left_hand_rz, mass 1e-10
- added link left_hip_rx, mass 1e-10
- added link left_shoulder_rz, mass 1e-10
- added link right_hand_rz, mass 1e-10
- added link right_hip_rz, mass 1e-10
- added link right_shoulder_rz, mass 1e-10
- link chest: mass 4 -> 3; geometry visual mesh filename=../../../model/panda/meshes/visual/chest_ascii.obj
- link head: geometry visual mesh filename=../../../model/panda/meshes/visual/head_ascii.obj
- link left_calf: mass 4 -> 3; geometry visual mesh filename=../../../model/panda/meshes/visual/calf.obj
- link left_foot: mass 4 -> 2; geometry visual mesh filename=../../../model/panda/meshes/visual/foot.obj
- link left_hand: geometry visual mesh filename=../../../model/panda/meshes/visual/hand_ascii.obj
- link left_lower_arm: geometry visual mesh filename=../../../model/panda/meshes/visual/lowerArm_ascii.obj
- link left_thigh: mass 4 -> 3; geometry visual mesh filename=../../../model/panda/meshes/visual/thigh.obj
- link left_upper_arm: geometry visual mesh filename=../../../model/panda/meshes/visual/upperArm_ascii.obj
- link right_calf: geometry visual mesh filename=../../../model/panda/meshes/visual/calf.obj
- link right_hand: geometry visual mesh filename=../../../model/panda/meshes/visual/hand_ascii.obj
- link right_lower_arm: geometry visual mesh filename=../../../model/panda/meshes/visual/lowerArm_ascii.obj
- link right_thigh: mass 4 -> 3; geometry visual mesh filename=../../../model/panda/meshes/visual/thigh.obj
- link right_upper_arm: geometry visual mesh filename=../../../model/panda/meshes/visual/upperArm_ascii.obj
Joints:
- removed joint j1
- removed joint j10
- removed joint j11
- removed joint j12
- removed joint j13
- removed joint j14
- removed joint j15
- removed joint j16
- removed joint j17
- removed joint j18
- removed joint j19
- removed joint j2
- removed joint j20
- removed joint j21
- removed joint j22
- removed joint j23
- removed joint j24
- removed joint j25
- removed joint j26
- removed joint j27
- removed joint j28
- removed joint j29
- removed joint j3
- removed joint j30
- removed joint j4
- removed joint j5
- removed joint j6
- removed joint j7
- removed joint j8
- removed joint j9
- added joint joint1: type revolute, parent right_foot, child right_calf, origin xyz=-0.06, 0, -0.8 rpy=0 0 0, axis 1 0 0, limit lower=-2.8973 upper=2.8973 effort=87 velocity=2.1750
- added joint joint10: type revolute, parent left_shoulder_ry, child left_upper_arm, origin xyz=0 0 0 rpy=0 0 0, axis 0 0 1, limit lower=-2.8973 upper=2.8973 effort=12 velocity=2.6100
- added joint joint11: type revolute, parent left_upper_arm, child left_lower_arm, origin xyz=0 0 0 rpy=0 0 0, axis 1 0 0, limit lower=-2.8973 upper=2.8973 effort=12 velocity=2.6100
- added joint joint12: type revolute, parent left_hand_ry, child left_hand, origin xyz=0 0 0 rpy=0 0 0, axis 0 0 1, limit lower=-2.8973 upper=2.8973 effort=12 velocity=2.6100
- added joint joint2: type revolute, parent right_calf, child right_thigh, origin xyz=0 0 0 rpy=0 0 0, axis 1 0 0, limit lower=-1.7628 upper=1.7628 effort=87 velocity=2.1750
- added joint joint3: type revolute, parent right_hip_ry, child chest, origin xyz=0 0 0 rpy=0 0 0, axis 0 0 1, limit lower=-2.8973 upper=2.8973 effort=87 velocity=2.1750
- added joint joint4: type revolute, parent left_hip_ry, child left_thigh, origin xyz=0 0 0 rpy=0 0 0, axis 1 0 0, limit lower=-3.0718 upper=-0.0698 effort=87 velocity=2.1750
- added joint joint5: type revolute, parent left_thigh, child left_calf, origin xyz=0 0 0 rpy=0 0 0, axis 1 0 0, limit lower=-2.8973 upper=2.8973 effort=12 velocity=2.6100
- added joint joint6: type revolute, parent left_calf, child left_foot, origin xyz=0 0 0 rpy=0 0 0, axis 1 0 0, limit lower=-0.0175 upper=3.7525 effort=12 velocity=2.6100
- added joint joint7: type revolute, parent right_shoulder_ry, child right_upper_arm, origin xyz=0 0 0 rpy=0 0 0, axis 0 0 1, limit lower=-2.8973 upper=2.8973 effort=12 velocity=2.6100
- added joint joint8: type revolute, parent right_upper_arm, child right_lower_arm, origin xyz=0 0 0 rpy=0 0 0, axis 1 0 0, limit lower=-2.8973 upper=2.8973 effort=12 velocity=2.6100
- added joint joint9: type revolute, parent right_hand_ry, child right_hand, origin xyz=0 0 0 rpy=0 0 0, axis 0 0 1, limit lower=-2.8973 upper=2.8973 effort=12 velocity=2.6100
