Commit message: backup with simulation loop update and prelim kinect task motion

File: model/human/human.urdf (robot description, URDF)
Before this commit: robot humann, 33 links, 32 joints
Links:
- removed link head_rx
- removed link head_ry
- removed link hip
- removed link hip_ry
- removed link hip_rz
- removed link left_foot_rx
- removed link left_foot_ry
- added link left_hand_rz, mass 1e-10
- added link left_hip_rx, mass 1e-10
- added link left_shoulder_rz, mass 1e-10
- added link right_hand_rz, mass 1e-10
- added link right_hip_rz, mass 1e-10
- added link right_shoulder_rz, mass 1e-10
- link chest: mass 4 -> 3; geometry visual mesh filename=../../../model/panda/meshes/visual/chest_ascii.obj
- link head: geometry visual mesh filename=../../../model/panda/meshes/visual/head_ascii.obj
- link left_calf: mass 4 -> 3; geometry visual mesh filename=../../../model/panda/meshes/visual/calf.obj
- link left_foot: mass 4 -> 2; geometry visual mesh filename=../../../model/panda/meshes/visual/foot.obj
- link left_hand: geometry visual mesh filename=../../../model/panda/meshes/visual/hand_ascii.obj
- link left_lower_arm: geometry visual mesh filename=../../../model/panda/meshes/visual/lowerArm_ascii.obj
- link left_thigh: mass 4 -> 3; geometry visual mesh filename=../../../model/panda/meshes/visual/thigh.obj
- link left_upper_arm: geometry visual mesh filename=../../../model/panda/meshes/visual/upperArm_ascii.obj
- link right_calf: geometry visual mesh filename=../../../model/panda/meshes/visual/calf.obj
- link right_foot: geometry visual mesh filename=../../../model/stanbot/meshes/visual/foot.obj
- link right_hand: geometry visual mesh filename=../../../model/panda/meshes/visual/hand_ascii.obj
- link right_lower_arm: geometry visual mesh filename=../../../model/panda/meshes/visual/lowerArm_ascii.obj
- link right_thigh: mass 4 -> 3; geometry visual mesh filename=../../../model/panda/meshes/visual/thigh.obj
- link right_upper_arm: geometry visual mesh filename=../../../model/panda/meshes/visual/upperArm_ascii.obj
Joints:
- removed joint left_ankle_1
- removed joint left_ankle_2
- removed joint left_ankle_3
- removed joint left_elbow
- removed joint left_hip_1
- removed joint left_hip_2
- removed joint left_hip_3
- removed joint left_knee
- removed joint left_shoulder_1
- removed joint left_shoulder_2
- removed joint left_shoulder_3
- removed joint left_wrist_1
- removed joint left_wrist_2
- removed joint left_wrist_3
- removed joint neck_1
- removed joint neck_2
- removed joint neck_3
- removed joint right_ankle
- removed joint right_elbow
- removed joint right_hip_1
- removed joint right_hip_2
- removed joint right_hip_3
- removed joint right_knee
- removed joint right_shoulder_1
- removed joint right_shoulder_2
- removed joint right_shoulder_3
- removed joint right_wrist_1
- removed joint right_wrist_2
- removed joint right_wrist_3
- removed joint waist_1
- removed joint waist_2
- removed joint waist_3
- added joint joint1: type revolute, parent right_foot, child right_calf, origin xyz=-0.06, 0, -0.8 rpy=0 0 0, axis 1 0 0, limit lower=-2.8973 upper=2.8973 effort=87 velocity=2.1750
- added joint joint10: type revolute, parent left_shoulder_ry, child left_upper_arm, origin xyz=0 0 0 rpy=0 0 0, axis 0 0 1, limit lower=-2.8973 upper=2.8973 effort=12 velocity=2.6100
- added joint joint11: type revolute, parent left_upper_arm, child left_lower_arm, origin xyz=0 0 0 rpy=0 0 0, axis 1 0 0, limit lower=-2.8973 upper=2.8973 effort=12 velocity=2.6100
- added joint joint12: type revolute, parent left_hand_ry, child left_hand, origin xyz=0 0 0 rpy=0 0 0, axis 0 0 1, limit lower=-2.8973 upper=2.8973 effort=12 velocity=2.6100
- added joint joint2: type revolute, parent right_calf, child right_thigh, origin xyz=0 0 0 rpy=0 0 0, axis 1 0 0, limit lower=-1.7628 upper=1.7628 effort=87 velocity=2.1750
- added joint joint3: type revolute, parent right_hip_ry, child chest, origin xyz=0 0 0 rpy=0 0 0, axis 0 0 1, limit lower=-2.8973 upper=2.8973 effort=87 velocity=2.1750
- added joint joint4: type revolute, parent left_hip_ry, child left_thigh, origin xyz=0 0 0 rpy=0 0 0, axis 1 0 0, limit lower=-3.0718 upper=-0.0698 effort=87 velocity=2.1750
- added joint joint5: type revolute, parent left_thigh, child left_calf, origin xyz=0 0 0 rpy=0 0 0, axis 1 0 0, limit lower=-2.8973 upper=2.8973 effort=12 velocity=2.6100
- added joint joint6: type revolute, parent left_calf, child left_foot, origin xyz=0 0 0 rpy=0 0 0, axis 1 0 0, limit lower=-0.0175 upper=3.7525 effort=12 velocity=2.6100
- added joint joint7: type revolute, parent right_shoulder_ry, child right_upper_arm, origin xyz=0 0 0 rpy=0 0 0, axis 0 0 1, limit lower=-2.8973 upper=2.8973 effort=12 velocity=2.6100
- added joint joint8: type revolute, parent right_upper_arm, child right_lower_arm, origin xyz=0 0 0 rpy=0 0 0, axis 1 0 0, limit lower=-2.8973 upper=2.8973 effort=12 velocity=2.6100
- added joint joint9: type revolute, parent right_hand_ry, child right_hand, origin xyz=0 0 0 rpy=0 0 0, axis 0 0 1, limit lower=-2.8973 upper=2.8973 effort=12 velocity=2.6100
