Commit message: controller update, stanbot joints renamed

File: template_project/stanbot.urdf (robot description, URDF)
Before this commit: robot stanbot, 31 links, 30 joints
Joints:
- removed joint j1
- removed joint j10
- removed joint j11
- removed joint j12
- removed joint j13
- removed joint j14
- removed joint j15
- removed joint j16
- removed joint j17
- removed joint j18
- removed joint j19
- removed joint j2
- removed joint j20
- removed joint j21
- removed joint j22
- removed joint j23
- removed joint j24
- removed joint j25
- removed joint j26
- removed joint j27
- removed joint j28
- removed joint j29
- removed joint j3
- removed joint j30
- removed joint j4
- removed joint j5
- removed joint j6
- removed joint j7
- removed joint j8
- removed joint j9
- added joint left_ankle_1: type revolute, parent left_calf, child left_foot_rx, origin xyz=0 0 -0.4 rpy=0 0 0, axis 1 0 0, limit lower=-0.0175 upper=3.7525 effort=12 velocity=2.6100
- added joint left_ankle_2: type revolute, parent left_foot_rx, child left_foot_ry, origin xyz=0 0 0 rpy=0 0 0, axis 0 1 0, limit lower=-0.0175 upper=3.7525 effort=12 velocity=2.6100
- added joint left_ankle_3: type revolute, parent left_foot_ry, child left_foot, origin xyz=0 0 0 rpy=0 0 0, axis 0 0 1, limit lower=-0.0175 upper=3.7525 effort=12 velocity=2.6100
- added joint left_elbow: type revolute, parent left_upper_arm, child left_lower_arm, origin xyz=0 0 -0.3 rpy=0 0 0, axis 1 0 0, limit lower=-2.8973 upper=2.8973 effort=12 velocity=2.6100
- added joint left_hip_1: type revolute, parent hip, child left_hip_rz, origin xyz=0.12 0 0 rpy=0 0 0, axis 0 0 1, limit lower=-3.0718 upper=-0.0698 effort=87 velocity=2.1750
- added joint left_hip_2: type revolute, parent left_hip_rz, child left_hip_ry, origin xyz=0 0 0 rpy=0 0 0, axis 0 1 0, limit lower=-3.0718 upper=-0.0698 effort=87 velocity=2.1750
- added joint left_hip_3: type revolute, parent left_hip_ry, child left_thigh, origin xyz=0 0 0 rpy=0 0 0, axis 1 0 0, limit lower=-3.0718 upper=-0.0698 effort=87 velocity=2.1750
- added joint left_knee: type revolute, parent left_thigh, child left_calf, origin xyz=0 0 -0.4 rpy=0 0 0, axis 1 0 0, limit lower=-2.8973 upper=2.8973 effort=12 velocity=2.6100
- added joint left_shoulder_1: type revolute, parent chest, child left_shoulder_rx, origin xyz=0.14 0 0.24 rpy=0 0 0, axis 1 0 0, limit lower=-2.8973 upper=2.8973 effort=12 velocity=2.6100
- added joint left_shoulder_2: type revolute, parent left_shoulder_rx, child left_shoulder_ry, origin xyz=0 0 0 rpy=0 0 0, axis 0 1 0, limit lower=-2.8973 upper=2.8973 effort=12 velocity=2.6100
- added joint left_shoulder_3: type revolute, parent left_shoulder_ry, child left_upper_arm, origin xyz=0 0 0 rpy=0 0 0, axis 0 0 1, limit lower=-2.8973 upper=2.8973 effort=12 velocity=2.6100
- added joint left_wrist_1: type revolute, parent left_lower_arm, child left_hand_rx, origin xyz=0 0 -0.3 rpy=0 0 0, axis 1 0 0, limit lower=-2.8973 upper=2.8973 effort=12 velocity=2.6100
- added joint left_wrist_2: type revolute, parent left_hand_rx, child left_hand_ry, origin xyz=0 0 0 rpy=0 0 0, axis 0 1 0, limit lower=-2.8973 upper=2.8973 effort=12 velocity=2.6100
- added joint left_wrist_3: type revolute, parent left_hand_ry, child left_hand, origin xyz=0 0 0 rpy=0 0 0, axis 0 0 1, limit lower=-2.8973 upper=2.8973 effort=12 velocity=2.6100
- added joint neck_1: type revolute, parent chest, child head_rx, origin xyz=0 0 0.30 rpy=0 0 0, axis 1 0 0, limit lower=-2.8973 upper=2.8973 effort=12 velocity=2.6100
- added joint neck_2: type revolute, parent head_rx, child head_ry, origin xyz=0 0 0 rpy=0 0 0, axis 0 1 0, limit lower=-2.8973 upper=2.8973 effort=12 velocity=2.6100
- added joint neck_3: type revolute, parent head_ry, child head, origin xyz=0 0 0 rpy=0 0 0, axis 0 0 1, limit lower=-2.8973 upper=2.8973 effort=12 velocity=2.6100
- added joint right_ankle: type revolute, parent right_foot, child right_calf, origin xyz=0 0.03 0.02 rpy=0 0 0, axis 1 0 0, limit lower=-2.8973 upper=2.8973 effort=87 velocity=2.1750
- added joint right_elbow: type revolute, parent right_upper_arm, child right_lower_arm, origin xyz=0 0 -0.3 rpy=0 0 0, axis 1 0 0, limit lower=-2.8973 upper=2.8973 effort=12 velocity=2.6100
- added joint right_hip_1: type revolute, parent right_thigh, child right_hip_rx, origin xyz=0 0 0.4 rpy=0 0 0, axis 1 0 0, limit lower=-2.8973 upper=2.8973 effort=87 velocity=2.1750
- added joint right_hip_2: type revolute, parent right_hip_rx, child right_hip_ry, origin xyz=0 0 0 rpy=0 0 0, axis 0 1 0, limit lower=-2.8973 upper=2.8973 effort=87 velocity=2.1750
- added joint right_hip_3: type revolute, parent right_hip_ry, child hip, origin xyz=0 0 0 rpy=0 0 0, axis 0 0 1, limit lower=-2.8973 upper=2.8973 effort=87 velocity=2.1750
- added joint right_knee: type revolute, parent right_calf, child right_thigh, origin xyz=0 0 0.4 rpy=0 0 0, axis 1 0 0, limit lower=-1.7628 upper=1.7628 effort=87 velocity=2.1750
- added joint right_shoulder_1: type revolute, parent chest, child right_shoulder_rx, origin xyz=-0.14 0 0.24 rpy=0 0 0, axis 1 0 0, limit lower=-2.8973 upper=2.8973 effort=12 velocity=2.6100
- added joint right_shoulder_2: type revolute, parent right_shoulder_rx, child right_shoulder_ry, origin xyz=0 0 0 rpy=0 0 0, axis 0 1 0, limit lower=-2.8973 upper=2.8973 effort=12 velocity=2.6100
- added joint right_shoulder_3: type revolute, parent right_shoulder_ry, child right_upper_arm, origin xyz=0 0 0 rpy=0 0 0, axis 0 0 1, limit lower=-2.8973 upper=2.8973 effort=12 velocity=2.6100
- added joint right_wrist_1: type revolute, parent right_lower_arm, child right_hand_rx, origin xyz=0 0 -0.3 rpy=0 0 0, axis 1 0 0, limit lower=-2.8973 upper=2.8973 effort=12 velocity=2.6100
- added joint right_wrist_2: type revolute, parent right_hand_rx, child right_hand_ry, origin xyz=0 0 0 rpy=0 0 0, axis 0 1 0, limit lower=-2.8973 upper=2.8973 effort=12 velocity=2.6100
- added joint right_wrist_3: type revolute, parent right_hand_ry, child right_hand, origin xyz=0 0 0 rpy=0 0 0, axis 0 0 1, limit lower=-2.8973 upper=2.8973 effort=12 velocity=2.6100
- added joint waist: type revolute, parent hip, child chest, origin xyz=0.06 0 0.2 rpy=0 0 0, axis 1 0 0, limit lower=-0.0175 upper=3.7525 effort=12 velocity=2.6100

Commit message: adjustments

File: template_project/stanbot.urdf (robot description, URDF)
Before this commit: robot stanbot, 33 links, 32 joints
Links:
- link chest: geometry visual mesh filename=../../../model/stanbot/meshes/visual/chest_ascii.obj; visual sphere radius=0.1

Commit message: new poses

File: template_project/stanbot.urdf (robot description, URDF)
Before this commit: robot stanbot, 33 links, 32 joints
Links:
- added link right_foot_ry, mass 1e-10
- link chest: geometry visual mesh filename=../../../model/stanbot/meshes/visual/chest_ascii.obj; visual sphere radius=0.05
Joints:
- removed joint left_ankle_1
- removed joint left_ankle_2
- removed joint left_ankle_3
- removed joint left_hip_1
- removed joint left_hip_2
- removed joint left_hip_3
- removed joint left_shoulder_1
- removed joint left_shoulder_2
- removed joint left_shoulder_3
- removed joint left_wrist_1
- removed joint left_wrist_2
- removed joint left_wrist_3
- removed joint right_ankle
- removed joint right_hip_1
- removed joint right_hip_2
- removed joint right_hip_3
- removed joint right_shoulder_1
- removed joint right_shoulder_2
- removed joint right_shoulder_3
- removed joint right_wrist_1
- removed joint right_wrist_2
- removed joint right_wrist_3
- removed joint waist_1
- removed joint waist_2
- removed joint waist_3
- added joint left_ankle_x: type revolute, parent left_calf, child left_foot_rx, origin xyz=0 0 -0.4 rpy=0 0 0, axis 1 0 0, limit lower=-0.0175 upper=3.7525 effort=12 velocity=2.6100
- added joint left_ankle_y: type revolute, parent left_foot_rx, child left_foot_ry, origin xyz=0 0 0 rpy=0 0 0, axis 0 1 0, limit lower=-0.0175 upper=3.7525 effort=12 velocity=2.6100
- added joint left_ankle_z: type revolute, parent left_foot_ry, child left_foot, origin xyz=0 0 0 rpy=0 0 0, axis 0 0 1, limit lower=-0.0175 upper=3.7525 effort=12 velocity=2.6100
- added joint left_hip_x: type revolute, parent left_hip_ry, child left_thigh, origin xyz=0 0 0 rpy=0 0 0, axis 1 0 0, limit lower=-3.0718 upper=-0.0698 effort=87 velocity=2.1750
- added joint left_hip_y: type revolute, parent left_hip_rz, child left_hip_ry, origin xyz=0 0 0 rpy=0 0 0, axis 0 1 0, limit lower=-3.0718 upper=-0.0698 effort=87 velocity=2.1750
- added joint left_hip_z: type revolute, parent hip, child left_hip_rz, origin xyz=0.12 0 0 rpy=0 0 0, axis 0 0 1, limit lower=-3.0718 upper=-0.0698 effort=87 velocity=2.1750
- added joint left_shoulder_x: type revolute, parent chest, child left_shoulder_rx, origin xyz=0.14 0 0.24 rpy=0 0 0, axis 1 0 0, limit lower=-2.8973 upper=2.8973 effort=12 velocity=2.6100
- added joint left_shoulder_y: type revolute, parent left_shoulder_rx, child left_shoulder_ry, origin xyz=0 0 0 rpy=0 0 0, axis 0 1 0, limit lower=-2.8973 upper=2.8973 effort=12 velocity=2.6100
- added joint left_shoulder_z: type revolute, parent left_shoulder_ry, child left_upper_arm, origin xyz=0 0 0 rpy=0 0 0, axis 0 0 1, limit lower=-2.8973 upper=2.8973 effort=12 velocity=2.6100
- added joint left_wrist_x: type revolute, parent left_lower_arm, child left_hand_rx, origin xyz=0 0 -0.3 rpy=0 0 0, axis 1 0 0, limit lower=-2.8973 upper=2.8973 effort=12 velocity=2.6100
- added joint left_wrist_y: type revolute, parent left_hand_rx, child left_hand_ry, origin xyz=0 0 0 rpy=0 0 0, axis 0 1 0, limit lower=-2.8973 upper=2.8973 effort=12 velocity=2.6100
- added joint left_wrist_z: type revolute, parent left_hand_ry, child left_hand, origin xyz=0 0 0 rpy=0 0 0, axis 0 0 1, limit lower=-2.8973 upper=2.8973 effort=12 velocity=2.6100
- added joint right_ankle_x: type revolute, parent right_foot_ry, child right_calf, origin xyz=0 0 0 rpy=0 0 0, axis 1 0 0, limit lower=-2.8973 upper=2.8973 effort=87 velocity=2.1750
- added joint right_ankle_y: type revolute, parent right_foot, child right_foot_ry, origin xyz=0 0.03 0.02 rpy=0 0 0, axis 0 1 0, limit lower=-2.8973 upper=2.8973 effort=87 velocity=2.1750
- added joint right_hip_x: type revolute, parent right_thigh, child right_hip_rx, origin xyz=0 0 0.4 rpy=0 0 0, axis 1 0 0, limit lower=-2.8973 upper=2.8973 effort=87 velocity=2.1750
- added joint right_hip_y: type revolute, parent right_hip_rx, child right_hip_ry, origin xyz=0 0 0 rpy=0 0 0, axis 0 1 0, limit lower=-2.8973 upper=2.8973 effort=87 velocity=2.1750
- added joint right_hip_z: type revolute, parent right_hip_ry, child hip, origin xyz=0 0 0 rpy=0 0 0, axis 0 0 1, limit lower=-2.8973 upper=2.8973 effort=87 velocity=2.1750
- added joint right_shoulder_x: type revolute, parent chest, child right_shoulder_rx, origin xyz=-0.14 0 0.24 rpy=0 0 0, axis 1 0 0, limit lower=-2.8973 upper=2.8973 effort=12 velocity=2.6100
- added joint right_shoulder_y: type revolute, parent right_shoulder_rx, child right_shoulder_ry, origin xyz=0 0 0 rpy=0 0 0, axis 0 1 0, limit lower=-2.8973 upper=2.8973 effort=12 velocity=2.6100
- added joint right_shoulder_z: type revolute, parent right_shoulder_ry, child right_upper_arm, origin xyz=0 0 0 rpy=0 0 0, axis 0 0 1, limit lower=-2.8973 upper=2.8973 effort=12 velocity=2.6100
- added joint right_wrist_x: type revolute, parent right_lower_arm, child right_hand_rx, origin xyz=0 0 -0.3 rpy=0 0 0, axis 1 0 0, limit lower=-2.8973 upper=2.8973 effort=12 velocity=2.6100
- added joint right_wrist_y: type revolute, parent right_hand_rx, child right_hand_ry, origin xyz=0 0 0 rpy=0 0 0, axis 0 1 0, limit lower=-2.8973 upper=2.8973 effort=12 velocity=2.6100
- added joint right_wrist_z: type revolute, parent right_hand_ry, child right_hand, origin xyz=0 0 0 rpy=0 0 0, axis 0 0 1, limit lower=-2.8973 upper=2.8973 effort=12 velocity=2.6100
- added joint waist_x: type revolute, parent hip_rz, child chest, origin xyz=0.0 0 0.0 rpy=0 0 0, axis 1 0 0, limit lower=-0.0175 upper=3.7525 effort=12 velocity=2.6100
- added joint waist_y: type revolute, parent hip, child hip_ry, origin xyz=0.0 0 0.2 rpy=0 0 0, axis 0 1 0, limit lower=-0.0175 upper=3.7525 effort=12 velocity=2.6100
- added joint waist_z: type revolute, parent hip_ry, child hip_rz, origin xyz=0.06 0 0.0 rpy=0 0 0, axis 0 0 1, limit lower=-0.0175 upper=3.7525 effort=12 velocity=2.6100

Commit message: working without progress and new poses

File: template_project/stanbot.urdf (robot description, URDF)
Before this commit: robot stanbot, 33 links, 32 joints
Links:
- added link right_foot_ry, mass 1e-10
Joints:
- added joint right_ankle_y: type revolute, parent right_foot, child right_foot_ry, origin xyz=0 0.0 0.0 rpy=0 0 0, axis 0 1 0, limit lower=-2.8973 upper=2.8973 effort=87 velocity=2.1750
- joint right_ankle: parent right_foot -> right_foot_ry
